Commit message: 0222_1519

File: legged_gym/resources/robots/hi_cl_23_240925/urdf/hi_cl_23_240925_rl.urdf (robot description, URDF)
Before this commit: robot hi_cl_23_240925, 24 links, 23 joints
Joints:
- joint l_ankle_pitch_joint: limit lower=-0.45 upper=1.15 effort=10 velocity=4 -> lower=-0.45 upper=1.15 effort=40 velocity=4
- joint l_ankle_roll_joint: limit lower=-0.15 upper=0.15 effort=10 velocity=4 -> lower=-0.15 upper=0.15 effort=40 velocity=4
- joint l_arm_roll_joint: limit lower=-3.14 upper=3.14 effort=10 velocity=4 -> lower=-3.14 upper=3.14 effort=40 velocity=4
- joint l_arm_yaw_joint: limit lower=-3.14 upper=3.14 effort=10 velocity=4 -> lower=-3.14 upper=3.14 effort=40 velocity=4
- joint l_calf_joint: limit lower=-0.8 upper=1.5 effort=10 velocity=4 -> lower=-0.8 upper=1.5 effort=40 velocity=4
- joint l_hip_pitch_joint: limit lower=-1.0 upper=1.8 effort=10 velocity=4 -> lower=-1.0 upper=1.8 effort=40 velocity=4
- joint l_hip_roll_joint: limit lower=-0.12 upper=0.5 effort=10 velocity=4 -> lower=-0.12 upper=0.5 effort=40 velocity=4
- joint l_shoulder_pitch_joint: limit lower=-3.14 upper=3.14 effort=10 velocity=4 -> lower=-3.14 upper=3.14 effort=40 velocity=4
- joint l_shoulder_roll_joint: limit lower=-3.14 upper=3.14 effort=10 velocity=4 -> lower=-3.14 upper=3.14 effort=40 velocity=4
- joint l_thigh_joint: limit lower=-0.3 upper=0.6 effort=10 velocity=4 -> lower=-0.3 upper=0.6 effort=40 velocity=4
- joint l_wrist_yaw_joint: limit lower=-3.14 upper=3.14 effort=10 velocity=4 -> lower=-3.14 upper=3.14 effort=40 velocity=4
- joint loin_yaw_joint: limit lower=-3.14 upper=3.14 effort=10 velocity=4 -> lower=-3.14 upper=3.14 effort=40 velocity=4
- joint r_ankle_pitch_joint: limit lower=-0.45 upper=1.15 effort=10 velocity=4 -> lower=-0.45 upper=1.15 effort=40 velocity=4
- joint r_ankle_roll_joint: limit lower=-0.15 upper=0.15 effort=10 velocity=4 -> lower=-0.15 upper=0.15 effort=40 velocity=4
- joint r_arm_roll_joint: limit lower=-3.14 upper=3.14 effort=10 velocity=4 -> lower=-3.14 upper=3.14 effort=40 velocity=4
- joint r_arm_yaw_joint: limit lower=-3.14 upper=3.14 effort=10 velocity=4 -> lower=-3.14 upper=3.14 effort=40 velocity=4
- joint r_calf_joint: limit lower=-0.8 upper=1.5 effort=10 velocity=4 -> lower=-0.8 upper=1.5 effort=40 velocity=4
- joint r_hip_pitch_joint: limit lower=-1.0 upper=1.8 effort=10 velocity=4 -> lower=-1.0 upper=1.8 effort=40 velocity=4
- joint r_hip_roll_joint: limit lower=-0.5 upper=0.12 effort=10 velocity=4 -> lower=-0.5 upper=0.12 effort=40 velocity=4
- joint r_shoulder_pitch_joint: limit lower=-3.14 upper=3.14 effort=10 velocity=4 -> lower=-3.14 upper=3.14 effort=40 velocity=4
- joint r_shoulder_roll_joint: limit lower=-3.14 upper=3.14 effort=10 velocity=4 -> lower=-3.14 upper=3.14 effort=40 velocity=4
- joint r_thigh_joint: limit lower=-0.6 upper=0.3 effort=10 velocity=4 -> lower=-0.6 upper=0.3 effort=40 velocity=4
- joint r_wrist_yaw_joint: limit lower=-3.14 upper=3.14 effort=10 velocity=4 -> lower=-3.14 upper=3.14 effort=40 velocity=4

Commit message: 0303_1001_

File: legged_gym/resources/robots/hi_cl_23_240925/urdf/hi_cl_23_240925_rl.urdf (robot description, URDF)
Before this commit: robot hi_cl_23_240925, 24 links, 23 joints
Joints:
- joint l_ankle_pitch_joint: origin xyz=0 0 -0.2 rpy=0 -0.55 0 -> xyz=0 0 -0.2 rpy=0 -0.25 0
- joint l_calf_joint: origin xyz=0 0 -0.10575 rpy=0 1.1 0 -> xyz=0 0 -0.10575 rpy=0 0.6 0
- joint l_hip_pitch_joint: origin xyz=0 0.02875 -0.06425 rpy=0 -0.55 0 -> xyz=0 0.02875 -0.06425 rpy=0 -0.35 0
- joint r_ankle_pitch_joint: origin xyz=0 0 -0.2 rpy=0 -0.55 0 -> xyz=0 0 -0.2 rpy=0 -0.25 0
- joint r_calf_joint: origin xyz=0 0 -0.10575 rpy=0 1.1 0 -> xyz=0 0 -0.10575 rpy=0 0.6 0
- joint r_hip_pitch_joint: origin xyz=0 -0.02875 -0.06425 rpy=0 -0.55 0 -> xyz=0 -0.02875 -0.06425 rpy=0 -0.35 0
